File: main1.brd (EAGLE design)
At the start: 87.6 x 40.6 mm, 17 parts, among them T1 THONKICONN, T2 THONKICONN

Commit message: Add files via upload
Parts:
- added JP2, JP5, JP6: (no value), _JC:1X03/OCT
- added U$1, U$2, U$3, U$4: (no value), _JC:HOLE_3MM
- moved JP4 23.2 mm to (82.5, 69.8), turned to 90 degrees
- moved JP1 18.4 mm to (43.8, 88.9)
- moved JP3 12.3 mm to (5.08, 62.2)
- moved CH2 2.54 mm to (11.4, 59.4)
- moved DIO1 2.54 mm to (45.7, 59.4)
- moved DIO3 2.54 mm to (55.9, 59.4)
- moved DIO5 2.54 mm to (66.0, 59.4)
- moved DIO7 2.54 mm to (76.2, 59.4)
- moved T2 2.54 mm to (34.3, 59.4)
- moved WG2 2.54 mm to (22.9, 59.4)
Connections:
- removed net CH1-: CH1.P3, JP1.P2
- removed net CH2-: CH2.P3, JP1.P4
- net CH1+: now also JP2.1
- net CH2+: now also JP2.2
- net GND: now also CH1.P3, CH2.P3, JP1.P2, JP1.P4, JP2.3, JP5.3, JP6.3
- net T1: now also JP6.1
- net T2: now also JP6.2
- net WG1: now also JP5.1
- net WG2: now also JP5.2
Routing:
- net DIO6: track 69.9 -> 22.7 mm
- net CH2-: track 25.7 -> 0.00 mm
- net DIO8: track 34.2 -> 59.5 mm
- net CH1-: track 22.0 -> 0.00 mm
- net DIO3: track 56.5 -> 36.3 mm
- net DIO5: track 61.6 -> 41.4 mm
- net DIO7: track 66.6 -> 46.5 mm
- net DIO9: track 35.0 -> 54.7 mm
- net DIO1: track 51.4 -> 33.3 mm
- net DIO4: track 35.7 -> 17.6 mm
- net DIO2: track 30.6 -> 12.6 mm
- net CH2+: track 37.2 -> 54.1 mm
- net CH1+: track 10.5 -> 26.6 mm
- net DIO0: track 26.8 -> 11.0 mm
- net DIO10: track 35.0 -> 50.0 mm
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Other:
- board size 87.6 x 40.6 mm -> 87.6 x 38.1 mm
- board text added: "C1"
- board text added: "C1/C2"
- board text added: "C2"
- board text added: "Digilent AD2 Interface Board Rev.a"
- board text added: "W1/W2"
- board text removed: "CH1/CH2"
- board text removed: "Digilent AD2 Synth IO Rev.a"
- board text removed: "WG1/WG2"
